Commit message: front and back cam added

File: fb_description/urdf/fb.xacro (robot description, xacro)
@@ -59,5 +59,10 @@
     <parent link="chassis"/>
     <child link="camera_link"/>
-  </joint>
+</joint>
+   <joint name="camera_back_joint" type="fixed">
+    <origin xyz="-0.22 0.0 0.04" rpy="0 0 -3.14"/>
+    <parent link="chassis"/>
+    <child link="camera_back_link"/>
+</joint>
   <link name="camera_link">
     <visual>
@@ -82,4 +87,26 @@
     </inertial>-->
   </link>
+  <link name="camera_back_link">
+    <visual>
+     <origin xyz="0 0 0" rpy="1.57 1.57 1.57"/>
+     <geometry>
+        <box size="0.012 0.132 0.020"/>
+      </geometry>
+   </visual>
+    <collision>
+      <origin xyz="0.003 0.065 0.007" rpy="0 0 0"/>
+      <geometry>
+        <box size="0.012 0.132 0.020"/>
+      </geometry>
+    </collision>
+    <!-- This inertial field needs doesn't contain reliable data!! -->
+<!--   <inertial>
+      <mass value="0.564" />
+      <origin xyz="0 0 0" />
+      <inertia ixx="0.003881243" ixy="0.0" ixz="0.0"
+               iyy="0.000498940" iyz="0.0"
+               izz="0.003879257" />
+    </inertial>-->
+  </link>
   <joint name="camera_rgb_joint" type="fixed">
     <origin xyz="${r200_cam_rgb_px} ${r200_cam_rgb_py} ${r200_cam_rgb_pz}" rpy="0 0 0"/>
